Commit message: Chnge the tarsus joint to fixed because we do not need it

File: urdf/hexapod_model.xacro (robot description, xacro)
@@ -284,5 +284,5 @@
         </gazebo>
         <!-- tarsus -->
-        <joint name="tarsus_joint_${side}${position}" type="revolute">
+        <joint name="tarsus_joint_${side}${position}" type="fixed">
             <origin xyz="${tibia_length} 0.0 0.0" rpy="0.0 0.0 0.0"/>
             <parent link="tibia_${side}${position}"/>
@@ -291,14 +291,4 @@
             <limit lower="${joint_lower_limit}" upper="${joint_upper_limit}" effort="${joint_effort}" velocity="${joint_velocity}"/>
         </joint>
-        <transmission name="tarsus_transmission_${side}${position}">
-            <type>transmission_interface/SimpleTransmission</type>
-            <joint name="tarsus_joint_${side}${position}">
-                <hardwareInterface>hardware_interface/EffortJointInterface</hardwareInterface>
-            </joint>
-            <actuator name="tarsus_motor_${side}${position}">
-                <hardwareInterface>hardware_interface/EffortJointInterface</hardwareInterface>
-                <mechanicalReduction>1</mechanicalReduction>
-            </actuator>
-        </transmission>
         <link name="tarsus_${side}${position}">
             <visual>
